File: JAE/test board.brd (EAGLE design)
At the start: 92.4 x 130.8 mm, 2 parts

Commit message: test 3
Parts:
- moved BQ78350-R1 7.18 mm to (6.35, 8.89)
Routing:
- net N$3: track 23.6 -> 30.8 mm
- net N$1: track 88.8 -> 96.0 mm
Changed lines of the file:
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@@
 <attribute name="VALUE" x="35.7124" y="11.0744" size="3.175" layer="27"/>
 </element>
-<element name="BQ78350-R1" library="Hydro-Common-Comp" package="TSSOP-30" package3d_urn="urn:adsk.eagle:package:6217949/2" value="BQ78350-R1" x="11.43" y="13.97" smashed="yes">
-<attribute name="NAME" x="10.524884375" y="12.395040625" size="2.299" layer="21" rot="R90"/>
-<attribute name="NAME" x="11.43" y="24.2582" size="0.662709375" layer="25"/>
-<attribute name="VALUE" x="11.43" y="12.7999" size="0.668646875" layer="27" align="top-left"/>
+<element name="BQ78350-R1" library="Hydro-Common-Comp" package="TSSOP-30" package3d_urn="urn:adsk.eagle:package:6217949/2" value="BQ78350-R1" x="6.35" y="8.89" smashed="yes">
+<attribute name="NAME" x="5.444884375" y="7.315040625" size="2.299" layer="21" rot="R90"/>
+<attribute name="NAME" x="6.35" y="19.1782" size="0.662709375" layer="25"/>
+<attribute name="VALUE" x="6.35" y="7.7199" size="0.668646875" layer="27" align="top-left"/>
 </element>
 </elements>
@@
 <contactref element="BAT1" pad="P$1"/>
 <contactref element="BQ78350-R1" pad="P$20"/>
-<wire x1="16.4592" y1="18.8976" x2="16.4592" y2="19.3548" width="0.1524" layer="1"/>
-<wire x1="16.764" y1="18.5928" x2="16.4592" y2="18.8976" width="0.1524" layer="1"/>
-<wire x1="37.1856" y1="18.5928" x2="16.764" y2="18.5928" width="0.1524" layer="1"/>
-<wire x1="38.7096" y1="20.1168" x2="37.1856" y2="18.5928" width="0.1524" layer="1"/>
-<wire x1="16.4592" y1="19.3548" x2="16.43" y2="19.37" width="0.1524" layer="1"/>
+<wire x1="11.3792" y1="13.8176" x2="11.3792" y2="14.2748" width="0.1524" layer="1"/>
+<wire x1="11.684" y1="13.5128" x2="11.3792" y2="13.8176" width="0.1524" layer="1"/>
+<wire x1="32.1056" y1="13.5128" x2="11.684" y2="13.5128" width="0.1524" layer="1"/>
+<wire x1="38.7096" y1="20.1168" x2="32.1056" y2="13.5128" width="0.1524" layer="1"/>
+<wire x1="11.3792" y1="14.2748" x2="11.35" y2="14.29" width="0.1524" layer="1"/>
 <wire x1="38.7096" y1="20.1168" x2="38.7858" y2="20.2438" width="0.1524" layer="1"/>
 </signal>
@@
 <contactref element="BAT1" pad="P$2"/>
 <contactref element="BQ78350-R1" pad="P$16"/>
-<wire x1="18.4404" y1="79.4004" x2="18.4404" y2="19.5072" width="0.1524" layer="1"/>
-<wire x1="38.7096" y1="99.6696" x2="18.4404" y2="79.4004" width="0.1524" layer="1"/>
-<wire x1="18.4404" y1="19.5072" x2="18.43" y2="19.37" width="0.1524" layer="1"/>
+<wire x1="13.3604" y1="74.3204" x2="13.3604" y2="14.4272" width="0.1524" layer="1"/>
+<wire x1="38.7096" y1="99.6696" x2="13.3604" y2="74.3204" width="0.1524" layer="1"/>
+<wire x1="13.3604" y1="14.4272" x2="13.35" y2="14.29" width="0.1524" layer="1"/>
 <wire x1="38.7096" y1="99.6696" x2="38.7858" y2="99.6696" width="0.1524" layer="1"/>
 </signal>

Commit message: saved
Routing:
- net N$3: track 30.8 -> 54.7 mm
Changed lines of the file:
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@@
 <contactref element="BAT1" pad="P$1"/>
 <contactref element="BQ78350-R1" pad="P$20"/>
-<wire x1="11.3792" y1="13.8176" x2="11.3792" y2="14.2748" width="0.1524" layer="1"/>
-<wire x1="11.684" y1="13.5128" x2="11.3792" y2="13.8176" width="0.1524" layer="1"/>
-<wire x1="32.1056" y1="13.5128" x2="11.684" y2="13.5128" width="0.1524" layer="1"/>
-<wire x1="38.7096" y1="20.1168" x2="32.1056" y2="13.5128" width="0.1524" layer="1"/>
-<wire x1="11.3792" y1="14.2748" x2="11.35" y2="14.29" width="0.1524" layer="1"/>
+<wire x1="4.90735" y1="15.854896875" x2="4.90734375" y2="15.85489375" width="0.1524" layer="1"/>
+<wire x1="4.90734375" y1="15.85489375" x2="4.984546875" y2="10.04513125" width="0.1524" layer="1"/>
+<wire x1="4.984546875" y1="10.04513125" x2="5.15659375" y2="8.67556875" width="0.1524" layer="1"/>
+<wire x1="4.90735" y1="15.854896875" x2="11.35" y2="15.65964375" width="0.1524" layer="1"/>
+<wire x1="5.15659375" y1="8.67556875" x2="6.650909375" y2="7.1628" width="0.1524" layer="1"/>
+<wire x1="6.650909375" y1="7.1628" x2="25.7556" y2="7.1628" width="0.1524" layer="1"/>
+<wire x1="11.35" y1="15.65964375" x2="11.35" y2="14.29" width="0.1524" layer="1"/>
+<wire x1="38.7096" y1="20.1168" x2="25.7556" y2="7.1628" width="0.1524" layer="1"/>
 <wire x1="38.7096" y1="20.1168" x2="38.7858" y2="20.2438" width="0.1524" layer="1"/>
 </signal>
